File: Hardware/Spectroscilloscope Revised_2.brd (EAGLE design)
At the start: 160 x 100 mm, 52 parts, among them IC1 7805TV, Q1 16MHz, U1 ATMEGA328P-PU, U2 MCP6024-I/P, U3 MCP6024-I/P

Commit message: Wroked on PCB, updated Schematic
Parts:
- added CAPTURING, POWER: (no value), led:LED5MM
- added R12, R13: 330, rcl:0204/7
- C10, C8, C9: device capacitor-wima:C2.5-3 -> rcl:C050-024X044
- moved O2CAL 232.7 mm to (47.0, 161.3)
- moved O1CAL 221.5 mm to (36.8, 161.3)
- moved 0.23CAL 205.2 mm to (26.7, 161.3)
- moved 2.5CAL 204.7 mm to (16.5, 161.3)
- moved C3 163.3 mm to (58.4, 154.9), turned to 180 degrees
- moved 12VPOWER 151.9 mm to (31.8, 170.2), turned to 180 degrees
- moved SPST 140.5 mm to (17.8, 170.2)
- moved C2 139.0 mm to (58.4, 161.3)
- moved C15 137.5 mm to (58.4, 167.6)
- moved D2 136.8 mm to (43.2, 132.1), turned to 90 degrees
- moved C5 136.8 mm to (58.4, 141.0)
- moved HC05 136.4 mm to (54.6, 101.6)
- moved PROBESELECT 135.6 mm to (38.1, 104.1)
- moved D1 133.1 mm to (50.8, 132.1), turned to 90 degrees
- moved C16 132.1 mm to (58.4, 133.3)
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Connections:
- removed net N$11: R8.2, U1.3
- new net N$12: POWER.K, R12.2
- new net N$13: CAPTURING.K, R13.2
- new net N$14: CAPTURING.A, U1.6
- net GND: now also R12.1, R13.1
- net VCC: now also POWER.A
Routing:
- net VCC: track 0.00 -> 358.2 mm
- net VREF_O1: track 0.00 -> 182.2 mm, vias 0 -> 1
- net N$7: track 0.00 -> 180.1 mm
- net 2.5VREF: track 0.00 -> 179.6 mm, vias 0 -> 2
- net VIN: track 0.00 -> 154.5 mm, vias 0 -> 1
- net N$10: track 0.00 -> 134.0 mm, vias 0 -> 1
- net N$3: track 0.00 -> 132.6 mm
- net NONINV: track 0.00 -> 128.1 mm, vias 0 -> 1
- net 0.23VREF: track 0.00 -> 127.5 mm, vias 0 -> 1
- net X10: track 0.00 -> 125.3 mm, vias 0 -> 1
- net +12V: track 0.00 -> 123.8 mm, vias 0 -> 1
- net X1: track 0.00 -> 123.5 mm, vias 0 -> 1
- net N$8: track 0.00 -> 111.9 mm, vias 0 -> 1
- net VREF_O2: track 0.00 -> 111.0 mm, vias 0 -> 2
- net N$13: track 0.00 -> 107.5 mm, vias 0 -> 1
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- added copper zone on layer 16, net GND
Other:
- board size 160 x 100 mm -> 68.6 x 150.2 mm
- board text added: "Alick Campbell ECNG3020 University of the West Indies, Mona"
- board text added: "Spectroscilloscope"

Commit message: Updated Schematics
Parts:
- added PROBECON: (no value), pinhead:2X03
- moved CAPTURING 4.10 mm to (53.8, 44.0)
Connections:
- net +12VI: now also 12VPOWER.1; no longer 12VPOWER.2, 12VPOWER.3
- net GND: now also 12VPOWER.2, 12VPOWER.3, PROBECON.1, PROBECON.2, PROBECON.3, PROBECON.4, PROBECON.5; no longer 12VPOWER.1
- net VIN: now also PROBECON.6
Routing:
- net N$9: track 96.6 -> 149.5 mm, vias 0 -> 1
- net VREF_O2: track 111.0 -> 151.8 mm, vias 2 -> 1
- net N$10: track 134.0 -> 160.9 mm, vias 1 -> 2
- net X10: track 125.3 -> 148.5 mm, vias 1 -> 0
- net +12V: track 123.8 -> 142.6 mm
- net VREF_O1: track 182.2 -> 163.7 mm
- net NONINV: track 128.1 -> 144.5 mm, vias 1 -> 2
- net VIN: track 154.5 -> 169.5 mm
- net N$13: track 107.5 -> 93.0 mm
- net N$3: track 132.6 -> 118.3 mm, vias 0 -> 2
- net N$5: track 42.7 -> 56.8 mm, vias 2 -> 1
- net RST: track 69.5 -> 58.1 mm
- net TX: track 65.2 -> 55.0 mm, vias 1 -> 0
- net N$14: track 106.0 -> 96.2 mm, vias 1 -> 0
- net N$12: track 85.5 -> 78.7 mm
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Other:
- board text removed: "Spectroscilloscope"

Commit message: Revised the Front end design - Final revision - multisim simulation works - Testing Breadboard April 21
Connections:
- new net N$11: R3.1, R4.2
- new net N$17: R8.2, U1.24
- net NONINV: no longer R3.1, R4.2
- net TX: now also U1.23; no longer U1.2
Routing:
- net N$17: track 0.00 -> 46.3 mm
- net TX: track 55.0 -> 59.9 mm, vias 0 -> 2
- net N$11: track 0.00 -> 2.54 mm
- net NONINV: track 144.5 -> 142.1 mm
Changed lines of the file:
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@@
 <setting verticaltext="up"/>
 </settings>
-<grid distance="0.003333" unitdist="inch" unit="inch" style="lines" multiple="1" display="yes" altdistance="5" altunitdist="mil" altunit="mm"/>
+<grid distance="0.003333" unitdist="inch" unit="mil" style="lines" multiple="1" display="yes" altdistance="5" altunitdist="mil" altunit="mil"/>
 <layers>
 <layer number="1" name="Top" color="4" fill="1" visible="yes" active="yes"/>
@@
 ECNG3020
 University of the West Indies, Mona</text>
+<dimension x1="2.54" y1="31.75" x2="2.54" y2="182" x3="-35.641103125" y3="106.875" textsize="1.778" layer="1"/>
+<dimension x1="2.54" y1="181.991" x2="71.12" y2="181.991" x3="36.83" y3="196.914971875" textsize="1.778" layer="1"/>
 </plain>
 <attributes>
@@
 <contactref element="C5" pad="2"/>
 <contactref element="C4" pad="1"/>
-<contactref element="R4" pad="2"/>
-<contactref element="R3" pad="1"/>
 <contactref element="R6" pad="2"/>
 <wire x1="60.96" y1="135.89" x2="50.8" y2="135.89" width="0.4064" layer="1"/>
@@
 <wire x1="60.96" y1="140.97" x2="60.96" y2="143.51" width="0.4064" layer="1"/>
 <wire x1="31.75" y1="100.33" x2="30.48" y2="99.06" width="0.4064" layer="1"/>
-<wire x1="31.75" y1="115.2525" x2="31.75" y2="100.33" width="0.4064" layer="1"/>
+<wire x1="31.75" y1="115.2525" x2="31.75" y2="114.935" width="0.4064" layer="1"/>
+<wire x1="31.75" y1="114.935" x2="31.75" y2="100.33" width="0.4064" layer="1"/>
 <wire x1="30.48" y1="116.5225" x2="31.75" y2="115.2525" width="0.4064" layer="1"/>
-<wire x1="30.48" y1="142.24" x2="30.48" y2="116.5225" width="0.4064" layer="1"/>
-<wire x1="30.48" y1="142.24" x2="33.02" y2="142.24" width="0.4064" layer="1"/>
 <wire x1="36.83" y1="134.62" x2="43.18" y2="128.27" width="0.4064" layer="1"/>
 <wire x1="36.83" y1="138.43" x2="36.83" y2="134.62" width="0.4064" layer="1"/>
-<wire x1="33.02" y1="142.24" x2="36.83" y2="138.43" width="0.4064" layer="1"/>
 <wire x1="19.685" y1="74.295" x2="15.24" y2="69.85" width="0.4064" layer="1"/>
 <wire x1="19.685" y1="85.725" x2="19.685" y2="74.295" width="0.4064" layer="1"/>
@@
 <via x="19.685" y="85.725" extent="1-16" drill="0.35"/>
 <via x="29.845" y="85.725" extent="1-16" drill="0.35"/>
+<wire x1="32.385" y1="138.43" x2="36.83" y2="138.43" width="0.4064" layer="1"/>
+<wire x1="31.75" y1="139.065" x2="32.385" y2="138.43" width="0.4064" layer="1"/>
+<wire x1="30.48" y1="139.065" x2="31.75" y2="139.065" width="0.4064" layer="1"/>
+<wire x1="30.48" y1="116.205" x2="30.48" y2="139.065" width="0.4064" layer="1"/>
+<wire x1="31.75" y1="114.935" x2="30.48" y2="116.205" width="0.4064" layer="1"/>
 </signal>
 <signal name="X1">
@@
 <signal name="TX">
 <contactref element="HC05" pad="3"/>
-<contactref element="U1" pad="2"/>
 <wire x1="39.6875" y1="98.1075" x2="53.34" y2="84.455" width="0.4064" layer="16"/>
 <wire x1="33.9725" y1="98.1075" x2="39.6875" y2="98.1075" width="0.4064" layer="16"/>
-<wire x1="25.4" y1="106.68" x2="33.9725" y2="98.1075" width="0.4064" layer="16"/>
+<wire x1="25.4" y1="106.68" x2="26.67" y2="105.41" width="0.4064" layer="16"/>
+<wire x1="26.67" y1="105.41" x2="33.9725" y2="98.1075" width="0.4064" layer="16"/>
 <wire x1="16.51" y1="106.68" x2="25.4" y2="106.68" width="0.4064" layer="16"/>
-<wire x1="10.16" y1="113.03" x2="16.51" y2="106.68" width="0.4064" layer="16"/>
+<contactref element="U1" pad="23"/>
+<wire x1="19.685" y1="100.965" x2="17.78" y2="102.87" width="0.4064" layer="16"/>
+<wire x1="24.765" y1="100.965" x2="19.685" y2="100.965" width="0.4064" layer="16"/>
+<wire x1="27.305" y1="103.505" x2="24.765" y2="100.965" width="0.4064" layer="1"/>
+<wire x1="27.305" y1="105.41" x2="27.305" y2="103.505" width="0.4064" layer="1"/>
+<wire x1="26.67" y1="105.41" x2="27.305" y2="105.41" width="0.4064" layer="16"/>
+<via x="24.765" y="100.965" extent="1-16" drill="0.35"/>
+<via x="27.305" y="105.41" extent="1-16" drill="0.35"/>
 </signal>
 <signal name="KEY">
@@
 <wire x1="52.3875" y1="44.1325" x2="52.48795625" y2="44.022265625" width="0.4064" layer="1"/>
 </signal>
+<signal name="N$11">
+<contactref element="R4" pad="2"/>
+<contactref element="R3" pad="1"/>
+<wire x1="30.48" y1="142.24" x2="33.02" y2="142.24" width="0.4064" layer="1"/>
+</signal>
+<signal name="N$17">
+<contactref element="R8" pad="2"/>
+<contactref element="U1" pad="24"/>
+<wire x1="30.48" y1="105.41" x2="30.48" y2="104.14" width="0.4064" layer="16"/>
+<wire x1="38.1" y1="105.41" x2="30.48" y2="105.41" width="0.4064" layer="16"/>
+<wire x1="40.005" y1="107.315" x2="38.1" y2="105.41" width="0.4064" layer="16"/>
+<wire x1="40.005" y1="110.49" x2="40.005" y2="107.315" width="0.4064" layer="16"/>
+<wire x1="26.035" y1="110.49" x2="40.005" y2="110.49" width="0.4064" layer="16"/>
+<wire x1="23.495" y1="107.95" x2="26.035" y2="110.49" width="0.4064" layer="16"/>
+<wire x1="22.225" y1="107.95" x2="23.495" y2="107.95" width="0.4064" layer="16"/>
+<wire x1="20.955" y1="109.22" x2="22.225" y2="107.95" width="0.4064" layer="16"/>
+<wire x1="17.145" y1="109.22" x2="20.955" y2="109.22" width="0.4064" layer="16"/>
+<wire x1="15.24" y1="107.315" x2="17.145" y2="109.22" width="0.4064" layer="16"/>
+<wire x1="15.24" y1="105.41" x2="15.24" y2="107.315" width="0.4064" layer="16"/>
+<wire x1="17.78" y1="105.41" x2="15.24" y2="105.41" width="0.4064" layer="16"/>
+</signal>
 </signals>
