File: Hardware/Spectroscilloscope Revised_3.sch (EAGLE design)
At the start: 52 parts, among them IC1 7805TV, Q1 16MHz, U1 ATMEGA328P-PU, U2 MCP6024-I/P, U3 MCP6024-I/P

Commit message: Revised the Front end design - Final revision - multisim simulation works - Testing Breadboard April 21
Parts:
- removed C7: 0.1u, rcl:C-EU050-024X044
- removed O2CAL: (no value), pinhead:PINHD-1X2
- removed VREF_O2: 100k, pot:TRIM_EU-B25P
- added 1.25CAL: (no value), pinhead:PINHD-1X2
- added 1.25VREF: 100k, pot:TRIM_EU-B25P
- added CAPTURING, POWER: (no value), led:LED5MM
- added PROBECON: (no value), pinhead:PINHD-2X3
- added R12, R13: 330, rcl:R-EU_0204/7
- added R14, R15, R16, R17: 1k, rcl:R-EU_0204/7
Connections:
- removed net N$11: R8.2, U1.PD1
- removed net NONINV: C4.1, C5.2, D1.A, D2.C, R3.1, R4.2, R6.2, U2.VINA+
- removed net VREF_O2: C16.2, O2CAL.1, U3.VIND-, U3.VOUTD
- new net 1.25VREF: 1.25CAL.1, C15.2, U2.VINA+, U3.VINC-, U3.VOUTC
- new net CAPTURING: CAPTURING.A, U1.PD4
- new net COMPANDED: C4.1, C5.2, D1.A, D2.C, R11.2, R3.1, R4.2, R5.2
- new net N$12: POWER.C, R12.2
- new net N$13: CAPTURING.C, R13.2
- new net N$15: R14.2, R15.2, U2.VINB-
- new net N$17: R8.2, U1.PC1
- new net N$21: R16.2, R17.2, U2.VIND-
- new net N$22: R16.1, R7.1, U2.VOUTC
- net +12VI: now also 12VPOWER.1; no longer 12VPOWER.2, 12VPOWER.3
- net 0.23VREF: now also U2.VINC+; no longer U2.VINB+
- net 2.5VREF: now also U2.VINB+, U2.VIND+; no longer C7.2, R4.1, U2.VINC+
- net GND: now also 1.25CAL.2, 1.25VREF.A, 12VPOWER.2, 12VPOWER.3, PROBECON.1, PROBECON.2, PROBECON.3, PROBECON.4, PROBECON.5, R12.1, R13.1, R4.1; no longer 12VPOWER.1, C7.1, O2CAL.2, VREF_O2.A
- net N$10: now also VREF_O1.S; no longer VREF_O2.S
- net N$16: now also R11.1, R7.2; no longer R11.2, R5.1
- net N$4: now also R14.1, R6.1, U2.VOUTA; no longer R5.2, R7.1, U2.VOUTB
- net N$5: now also R5.1, R6.2, U2.VINA-; no longer R6.1, R7.2, U2.VINB-
- net N$7: now also 1.25VREF.S; no longer VREF_O1.S
- net TX: now also U1.PC0; no longer U1.PD0
- net VCC: now also 1.25VREF.E, POWER.A; no longer VREF_O2.E
- net VIN: now also PROBECON.6
- net VREF_O1: now also C16.2, U3.VIND-, U3.VOUTD; no longer C15.2, U3.VINC-, U3.VOUTC
- net X1: now also R15.1, U2.VOUTB; no longer U2.VINA-, U2.VOUTA
- net X10: now also R17.1, U2.VOUTD; no longer R11.1, U2.VOUTC
Other:
- moved on the sheet: 0.23CAL, 0.23VREF, 12VPOWER, 2.5CAL, 2.5VREF, C13, C14, C15, C16, C4, C5, D1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
